Commit message: Bigger goal/pos spaces

File: gym_envs_rhoban/urdf/my_cube.urdf (robot description, URDF)
Before this commit: robot cube, 1 links, 0 joints
Links:
- link baseLink: mass 0.1 -> None; geometry collision box size=1 1e-4 1; visual mesh filename=meshes/cube.obj scale=1 1e-4 1

File: gym_envs_rhoban/urdf/plane/plane.urdf (robot description, URDF)
Before this commit: robot plane, 1 links, 0 joints
Links:
- link planeLink: mass .0 -> 0
