Commit message: Massive refactor of environments; Move old environments to separate module for backwards compat

File: gym_envs_rhoban/urdf/RR100/rr100.urdf (robot description, URDF)
Before this commit: robot chassis, 11 links, 10 joints
Links:
- link base_footprint: mass .1 -> 0.01
- link base_link: mass .1 -> 0.01
- link front_left_wheel_link: geometry collision cylinder length=0.095 radius=0.21; visual cylinder length=0.095 radius=0.21
- link front_right_wheel_link: geometry collision cylinder length=0.095 radius=0.21; visual cylinder length=0.095 radius=0.21
- link rear_left_wheel_link: geometry collision cylinder length=0.095 radius=0.21; visual cylinder length=0.095 radius=0.21
- link rear_right_wheel_link: geometry collision cylinder length=0.095 radius=0.21; visual cylinder length=0.095 radius=0.21
Joints:
- removed joint front_left_wheel
- removed joint front_right_wheel
- removed joint rear_left_wheel
- removed joint rear_right_wheel
- added joint front_left_wheel_joint: type continuous, parent front_left_steering, child front_left_wheel_link, origin xyz=0 0.0 0 rpy=0 0 0, axis 0 1 0
- added joint front_right_wheel_joint: type continuous, parent front_right_steering, child front_right_wheel_link, origin xyz=0 -0.0 0 rpy=0 0 0, axis 0 1 0
- added joint rear_left_wheel_joint: type continuous, parent rear_left_steering, child rear_left_wheel_link, origin xyz=0 0.0 0 rpy=0 0 0, axis 0 1 0
- added joint rear_right_wheel_joint: type continuous, parent rear_right_steering, child rear_right_wheel_link, origin xyz=0 -0.0 0 rpy=0 0 0, axis 0 1 0

File: gym_envs_rhoban/urdf/UR5_RR100/rr100_ur.urdf (robot description, URDF)
Before this commit: robot chassis, 27 links, 26 joints
Links:
- removed link front_left_wheel_link
- removed link front_right_wheel_link
- removed link inertial_link
- removed link rear_left_wheel_link
- removed link rear_right_wheel_link
- added link front_left_wheel, mass 3; collision cylinder length=0.095 radius=0.21; visual cylinder length=0.095 radius=0.21
- added link front_right_wheel, mass 3; collision cylinder length=0.095 radius=0.21; visual cylinder length=0.095 radius=0.21
- added link rear_left_wheel, mass 3; collision cylinder length=0.095 radius=0.21; visual cylinder length=0.095 radius=0.21
- added link rear_right_wheel, mass 3; collision cylinder length=0.095 radius=0.21; visual cylinder length=0.095 radius=0.21
- added link rslidar, mass 0.87; collision cylinder length=0.081 radius=0.061; visual cylinder length=0.081 radius=0.061
- link base_footprint: mass .1 -> 0.01
- link base_link: mass .1 -> 70; geometry collision box size=0.86 0.27 0.442; collision box size=0.89 0.404 0.069
- link front_left_steering: mass 5.0 -> 2
- link front_right_steering: mass 5.0 -> 2
- link rear_left_steering: mass 5.0 -> 2
- link rear_right_steering: mass 5.0 -> 2
- link ur_ee_link: mass 0 -> 0.01
Joints:
- removed joint base_footprint_joint
- removed joint front_left_wheel
- removed joint front_right_wheel
- removed joint inertial_joint
- removed joint rear_left_wheel
- removed joint rear_right_wheel
- added joint base_joint: type fixed, parent base_footprint, child base_link, origin xyz=0 0 0.32075 rpy=0 0 0
- added joint base_link_to_rslidar: type fixed, parent base_link, child rslidar, origin xyz=0 0 0.45 rpy=0 0 0
- added joint front_left_wheel_joint: type continuous, parent front_left_steering, child front_left_wheel, origin xyz=0 0 0 rpy=-1.5707963267948963 0 0, axis 0 0 1
- added joint front_right_wheel_joint: type continuous, parent front_right_steering, child front_right_wheel, origin xyz=0 0 0 rpy=-1.5707963267948963 0 0, axis 0 0 1
- added joint rear_left_wheel_joint: type continuous, parent rear_left_steering, child rear_left_wheel, origin xyz=0 0 0 rpy=-1.5707963267948963 0 0, axis 0 0 1
- added joint rear_right_wheel_joint: type continuous, parent rear_right_steering, child rear_right_wheel, origin xyz=0 0 0 rpy=-1.5707963267948963 0 0, axis 0 0 1
- joint front_left_steering_joint: limit lower=-0.57 upper=0.57 effort=10.0 velocity=3.14 -> lower=-0.57 upper=0.57 effort=1000.0 velocity=0.5; origin xyz=0.30 0.279 -0.11075 rpy=0 0 0 -> xyz=0.25 0.275 -0.1 rpy=0 0 0
- joint front_right_steering_joint: limit lower=-0.57 upper=0.57 effort=10.0 velocity=3.14 -> lower=-0.57 upper=0.57 effort=1000.0 velocity=0.5; origin xyz=0.30 -0.279 -0.11075 rpy=0 0 0 -> xyz=0.25 -0.275 -0.1 rpy=0 0 0
- joint rear_left_steering_joint: limit lower=-0.57 upper=0.57 effort=10.0 velocity=3.14 -> lower=-0.57 upper=0.57 effort=1000.0 velocity=0.5; origin xyz=-0.25 0.279 -0.11075 rpy=0 0 0 -> xyz=-0.25 0.275 -0.1 rpy=0 0 0
- joint rear_right_steering_joint: limit lower=-0.57 upper=0.57 effort=10.0 velocity=3.14 -> lower=-0.57 upper=0.57 effort=1000.0 velocity=0.5; origin xyz=-0.25 -0.279 -0.11075 rpy=0 0 0 -> xyz=-0.25 -0.275 -0.1 rpy=0 0 0
